File: AuxBoard/AuxBoard.kicad_sch (KiCad schematic)
At the start: 29 parts, among them J1 ATX-24, J10 MatBIn, J11 FanHeader, J2 RPI4B, J4 MatrixASupply, J5 MatrixBSupply, J6 BigLED, J7 MatAOut, J8 MatAIn, J9 MatBOut, Q1 DMMT5401, Q2 DMG2305UX, Q3 DMG2305UX, Q4 DMG2305UX, SW1 SW_DPST, U1 74AHC04

Commit message: Updates to the Aux Board PCB
Parts:
- Q2, Q3, Q4: symbol Simulation_SPICE:PMOS -> Tom's Parts:PMOS
Connections:
- net +12V: now also Q4.2 (S); no longer Q4.3 (S)
- net +5VP: now also Q3.3 (D); no longer Q3.1 (D)
- net 5VSB: now also Q3.2 (S); no longer Q3.3 (S)
- net 5VSwitch: now also Q3.1 (G), Q4.1 (G); no longer Q3.2 (G), Q4.2 (G)
- net 5V_Power: now also Q2.2 (S); no longer Q2.3 (S)
- net at Q1.4 (C2), R2.2: now also Q2.1 (G); no longer Q2.2 (G)
- net at PolyFuse5.1, Q1.6 (E1): now also Q2.3 (D); no longer Q2.1 (D)
- net at J11.2 (Pin_2): now also Q4.3 (D); no longer Q4.1 (D)
Changed lines of the file:
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@@
     )
   )
-  (symbol (lib_id "Simulation_SPICE:PMOS") (at 36.83 67.31 270) (mirror x) (unit 1)
-    (in_bom yes) (on_board yes) (dnp no)
-    (property "Reference" "Q3" (at 36.83 58.42 90)
-      (effects (font (size 1.27 1.27)))
-    )
-    (property "Value" "DMG2305UX" (at 36.83 60.96 90)
-      (effects (font (size 1.27 1.27)))
-    )
-    (property "Footprint" "Package_TO_SOT_SMD:SOT-23-3" (at 39.37 62.23 0)
-      (effects (font (size 1.27 1.27)) hide)
-    )
-    (property "Datasheet" "https://ngspice.sourceforge.io/docs/ngspice-manual.pdf" (at 24.13 67.31 0)
-      (effects (font (size 1.27 1.27)) hide)
-    )
-    (property "Sim.Device" "PMOS" (at 19.685 67.31 0)
-      (effects (font (size 1.27 1.27)) hide)
-    )
-    (property "Sim.Type" "VDMOS" (at 17.78 67.31 0)
-      (effects (font (size 1.27 1.27)) hide)
-    )
-    (property "Sim.Pins" "1=D 2=G 3=S" (at 21.59 67.31 0)
+  (symbol (lib_id "Tom's Parts:PMOS") (at 36.83 67.31 270) (mirror x) (unit 1)
+    (in_bom yes) (on_board yes) (dnp no)
+    (property "Reference" "Q3" (at 48.26 60.96 90)
+      (effects (font (size 1.27 1.27)))
+    )
+    (property "Value" "DMG2305UX" (at 50.8 72.39 90)
+      (effects (font (size 1.27 1.27)))
+    )
+    (property "Footprint" "Package_TO_SOT_SMD:SOT-23-3" (at 41.91 83.82 0)
+      (effects (font (size 1.27 1.27)) hide)
+    )
+    (property "Datasheet" "https://ngspice.sourceforge.io/docs/ngspice-manual.pdf" (at 19.05 74.93 0)
+      (effects (font (size 1.27 1.27)) hide)
+    )
+    (property "Sim.Device" "PMOS" (at 34.29 86.36 0)
+      (effects (font (size 1.27 1.27)) hide)
+    )
+    (property "Sim.Type" "VDMOS" (at 36.83 86.36 0)
+      (effects (font (size 1.27 1.27)) hide)
+    )
+    (property "Sim.Pins" "1=S 2=D 3=G" (at 29.21 82.55 0)
       (effects (font (size 1.27 1.27)) hide)
     )
@@
     )
   )
-  (symbol (lib_id "Simulation_SPICE:PMOS") (at 130.81 111.76 270) (mirror x) (unit 1)
+  (symbol (lib_id "Tom's Parts:PMOS") (at 130.81 111.76 270) (mirror x) (unit 1)
     (in_bom yes) (on_board yes) (dnp no) (fields_autoplaced)
     (property "Reference" "Q2" (at 130.81 102.87 90)
@@
       (effects (font (size 1.27 1.27)))
     )
-    (property "Footprint" "Package_TO_SOT_SMD:SOT-23-3" (at 133.35 106.68 0)
-      (effects (font (size 1.27 1.27)) hide)
-    )
-    (property "Datasheet" "https://ngspice.sourceforge.io/docs/ngspice-manual.pdf" (at 118.11 111.76 0)
-      (effects (font (size 1.27 1.27)) hide)
-    )
-    (property "Sim.Device" "PMOS" (at 113.665 111.76 0)
-      (effects (font (size 1.27 1.27)) hide)
-    )
-    (property "Sim.Type" "VDMOS" (at 111.76 111.76 0)
-      (effects (font (size 1.27 1.27)) hide)
-    )
-    (property "Sim.Pins" "1=D 2=G 3=S" (at 115.57 111.76 0)
+    (property "Footprint" "Package_TO_SOT_SMD:SOT-23-3" (at 135.89 128.27 0)
+      (effects (font (size 1.27 1.27)) hide)
+    )
+    (property "Datasheet" "https://ngspice.sourceforge.io/docs/ngspice-manual.pdf" (at 113.03 119.38 0)
+      (effects (font (size 1.27 1.27)) hide)
+    )
+    (property "Sim.Device" "PMOS" (at 128.27 130.81 0)
+      (effects (font (size 1.27 1.27)) hide)
+    )
+    (property "Sim.Type" "VDMOS" (at 130.81 130.81 0)
+      (effects (font (size 1.27 1.27)) hide)
+    )
+    (property "Sim.Pins" "1=S 2=D 3=G" (at 123.19 127 0)
       (effects (font (size 1.27 1.27)) hide)
     )
@@
     )
   )
-  (symbol (lib_id "Simulation_SPICE:PMOS") (at 116.84 36.83 270) (mirror x) (unit 1)
+  (symbol (lib_id "Tom's Parts:PMOS") (at 116.84 36.83 270) (mirror x) (unit 1)
     (in_bom yes) (on_board yes) (dnp no)
     (property "Reference" "Q4" (at 116.84 27.94 90)
@@
       (effects (font (size 1.27 1.27)))
     )
-    (property "Footprint" "Package_TO_SOT_SMD:SOT-23-3" (at 119.38 31.75 0)
-      (effects (font (size 1.27 1.27)) hide)
-    )
-    (property "Datasheet" "https://ngspice.sourceforge.io/docs/ngspice-manual.pdf" (at 104.14 36.83 0)
-      (effects (font (size 1.27 1.27)) hide)
-    )
-    (property "Sim.Device" "PMOS" (at 99.695 36.83 0)
-      (effects (font (size 1.27 1.27)) hide)
-    )
-    (property "Sim.Type" "VDMOS" (at 97.79 36.83 0)
-      (effects (font (size 1.27 1.27)) hide)
-    )
-    (property "Sim.Pins" "1=D 2=G 3=S" (at 101.6 36.83 0)
-      (effects (font (size 1.27 1.27)) hide)
-    )
+    (property "Footprint" "Package_TO_SOT_SMD:SOT-23-3" (at 121.92 53.34 0)
+      (effects (font (size 1.27 1.27)) hide)
+    )
+    (property "Datasheet" "https://ngspice.sourceforge.io/docs/ngspice-manual.pdf" (at 99.06 44.45 0)
+      (effects (font (size 1.27 1.27)) hide)
+    )
+    (property "Sim.Device" "PMOS" (at 114.3 55.88 0)
+      (effects (font (size 1.27 1.27)) hide)
+    )
+    (property "Sim.Type" "VDMOS" (at 116.84 55.88 0)
+      (effects (font (size 1.27 1.27)) hide)
+    )
+    (property "Sim.Pins" "1=S 2=D 3=G" (at 109.22 52.07 0)
+      (effects (font (size 1.27 1.27)) hide)
+    )
